Commit message: hello

File: assets/ur5/doosan_origin.urdf (robot description, URDF)
Before this commit: robot Doosan_loz, 7 links, 6 joints
Links:
- added link base, mass 0.0
- added link ee_link, mass 0.0; collision box size=0.01 0.01 0.01
- added link rotated_base_link, mass 0.0
- added link tool0, mass 0.0
- added link tool_tip, mass 0.0
- added link world
Joints:
- added joint base_link-base_fixed_joint: type fixed, parent Base_0, child base, origin xyz=0 0 0 rpy=0 0 -3.14159265359
- added joint ee_fixed_joint: type fixed, parent link6, child ee_link, origin xyz=0.0 0.0 0.0 rpy=0 0.0 0.0
- added joint rotated_base-base_fixed_joint: type fixed, parent rotated_base_link, child Base_0, origin xyz=0.0 0.0 0.0 rpy=0.0 0.0 3.141592653589793
- added joint tool0_fixed_joint-tool_tip: type fixed, parent tool0, child tool_tip, origin xyz=0 0 0.145 rpy=0 0 0
- added joint world_joint: type fixed, parent world, child rotated_base_link, origin xyz=0.0 0.0 0.0 rpy=0.0 0.0 0.0
- added joint wrist_3_link-tool0_fixed_joint: type fixed, parent link6, child tool0, origin xyz=0 0.0823 0 rpy=-1.57079632679 0 0

File: assets/ur5/test.urdf (robot description, URDF)
Before this commit: robot Doosan_loz, 2 links, 1 joints
Links:
- removed link forearm_link
- removed link upper_arm_link
- added link base_link, mass 4.0; collision mesh filename=assets/ur5/visual/base.stl; visual mesh filename=assets/ur5/visual/base.stl
- added link shoulder_link, mass 3.7; collision mesh filename=assets/ur5/visual/shoulder.stl; visual mesh filename=assets/ur5/visual/shoulder.stl
Joints:
- removed joint elbow_joint
- added joint shoulder_pan_joint: type revolute, parent base_link, child shoulder_link, origin xyz=0.0 0.0 0.089159 rpy=0.0 0.0 0.0, axis 0 0 1, limit lower=-6.28318530718 upper=6.28318530718 effort=150.0 velocity=3.15

Commit message: Oke

File: assets/ur5/doosan_origin.urdf (robot description, URDF)
Before this commit: robot Doosan_loz, 13 links, 12 joints
Joints:
- joint base_link-base_fixed_joint: origin xyz=0 0 0 rpy=0 0 -3.14159265359 -> xyz=0 0 0 rpy=0 0 0
- joint joint1: limit lower=-2.167 upper=2.167 effort=30 velocity=1.571 -> lower=-6.283185307 upper=6.283185307 effort=150.0 velocity=2.617993878; origin xyz=0 0 0.1525 rpy=0 0 0 -> xyz=0 0 0.136 rpy=0 0 0
- joint joint2: limit lower=-2.167 upper=2.167 effort=30 velocity=1.571 -> lower=-6.28318530718 upper=6.28318530718 effort=150.0 velocity=2.617993878
- joint joint3: limit lower=-2.617 upper=2.617 effort=30 velocity=1.571 -> lower=-2.617993878 upper=2.617993878 effort=150.0 velocity=3.141592654
- joint joint4: limit lower=-2.617 upper=2.617 effort=30 velocity=1.571 -> lower=-6.28318530718 upper=6.28318530718 effort=150.0 velocity=3.926990817
- joint joint5: limit lower=-2.617 upper=2.617 effort=30 velocity=1.571 -> lower=-6.28318530718 upper=6.28318530718 effort=150.0 velocity=3.926990817
- joint joint6: limit lower=-2.617 upper=2.617 effort=30 velocity=1.571 -> lower=-6.28318530718 upper=6.28318530718 effort=150.0 velocity=3.926990817
- joint tool0_fixed_joint-tool_tip: origin xyz=0 0 0.145 rpy=0 0 0 -> xyz=0 0 0 rpy=0 0 0
- joint wrist_3_link-tool0_fixed_joint: origin xyz=0 0.0823 0 rpy=-1.57079632679 0 0 -> xyz=0 0 0 rpy=0 0 0

File: assets/ur5/test.urdf (robot description, URDF)
Before this commit: robot Doosan_loz, 2 links, 1 joints
Links:
- removed link base_link
- removed link shoulder_link
- added link link6, mass 1.128; visual mesh filename=m0609_collision/MF0609_6_0.dae scale=0.001 0.001 0.001
- added link tool0, mass 0.0
Joints:
- removed joint shoulder_pan_joint
- added joint wrist_3_link-tool0_fixed_joint: type fixed, parent link6, child tool0, origin xyz=0 0.0823 0 rpy=-1.57079632679 0 0
